File: door-sensor/hw/door_sensor.sch (EAGLE design)
At the start: 10 parts, among them IC1 PRO-MINI

Commit message: did a load of stuff that I can't remember and hadn't committed for a while
Parts:
- added C2: 0.47uF, SparkFun-Capacitors:10UF-POLAR-RADIAL-2.5MM-25V-20%
- added R4: 100k, SparkFun-Resistors:100KOHM-HORIZ-1/4W-1%
- added R5: 300k, SparkFun-Resistors:RESISTORAXIAL-0.3
Connections:
- new net BATTO: C2.+, IC1.A0, R4.2, R5.1
- new net DHT0: IC1.D4
- new net RIRQ: IC1.D2, NRF24L01+.8
- net DHTO: no longer IC1.D2
- net GND: now also C2.-, R4.1
- net VCC: now also R5.2
Changed lines of the file:
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@@
 <part name="SUPPLY5" library="SparkFun-PowerSymbols" deviceset="VCC" device=""/>
 <part name="C4" library="SparkFun-Capacitors" deviceset="0.1UF" device="-KIT-EZ-50V-20%" value="0.1uF"/>
+<part name="C2" library="SparkFun-Capacitors" deviceset="10UF-POLAR" device="-RADIAL-2.5MM-25V-20%" value="0.47uF"/>
+<part name="R4" library="SparkFun-Resistors" deviceset="100KOHM" device="-HORIZ-1/4W-1%" value="100k"/>
+<part name="SUPPLY6" library="SparkFun-PowerSymbols" deviceset="VCC" device=""/>
+<part name="GND6" library="SparkFun-PowerSymbols" deviceset="GND" device=""/>
+<part name="R5" library="SparkFun-Resistors" deviceset="RESISTOR" device="AXIAL-0.3" value="300k"/>
 </parts>
 <sheets>
@@
 <instance part="SUPPLY5" gate="G$1" x="17.78" y="114.3" rot="R270"/>
 <instance part="C4" gate="G$1" x="55.88" y="78.74"/>
+<instance part="C2" gate="G$1" x="-20.32" y="73.66"/>
+<instance part="R4" gate="G$1" x="-33.02" y="71.12" rot="R90"/>
+<instance part="SUPPLY6" gate="G$1" x="-33.02" y="91.44"/>
+<instance part="GND6" gate="1" x="-33.02" y="60.96"/>
+<instance part="R5" gate="G$1" x="-33.02" y="83.82" rot="R90"/>
 </instances>
 <busses>
@@
 <wire x1="15.24" y1="116.84" x2="15.24" y2="119.38" width="0.1524" layer="91"/>
 <wire x1="15.24" y1="119.38" x2="17.78" y2="119.38" width="0.1524" layer="91"/>
+</segment>
+<segment>
+<pinref part="R4" gate="G$1" pin="1"/>
+<pinref part="GND6" gate="1" pin="GND"/>
+<wire x1="-33.02" y1="66.04" x2="-33.02" y2="63.5" width="0.1524" layer="91"/>
+<pinref part="C2" gate="G$1" pin="-"/>
+<wire x1="-33.02" y1="66.04" x2="-20.32" y2="66.04" width="0.1524" layer="91"/>
+<wire x1="-20.32" y1="66.04" x2="-20.32" y2="68.58" width="0.1524" layer="91"/>
+<junction x="-33.02" y="66.04"/>
 </segment>
 </net>
@@
 <wire x1="12.7" y1="114.3" x2="17.78" y2="114.3" width="0.1524" layer="91"/>
 </segment>
+<segment>
+<pinref part="SUPPLY6" gate="G$1" pin="VCC"/>
+<wire x1="-33.02" y1="91.44" x2="-33.02" y2="88.9" width="0.1524" layer="91"/>
+<pinref part="R5" gate="G$1" pin="2"/>
+</segment>
 </net>
 <net name="SWO" class="0">
@@
 <net name="DHTO" class="0">
 <segment>
-<pinref part="IC1" gate="G$1" pin="D2"/>
-<wire x1="10.16" y1="17.78" x2="-7.62" y2="17.78" width="0.1524" layer="91"/>
-<label x="-7.62" y="17.78" size="1.778" layer="95" rot="R180" xref="yes"/>
-</segment>
-<segment>
 <pinref part="R2" gate="G$1" pin="2"/>
 <pinref part="DHT22" gate="G$1" pin="2"/>
@@
 </segment>
 </net>
+<net name="BATTO" class="0">
+<segment>
+<pinref part="R4" gate="G$1" pin="2"/>
+<wire x1="-33.02" y1="78.74" x2="-33.02" y2="76.2" width="0.1524" layer="91"/>
+<pinref part="C2" gate="G$1" pin="+"/>
+<wire x1="-33.02" y1="76.2" x2="-20.32" y2="76.2" width="0.1524" layer="91"/>
+<junction x="-33.02" y="76.2"/>
+<wire x1="-20.32" y1="76.2" x2="-20.32" y2="81.28" width="0.1524" layer="91"/>
+<junction x="-20.32" y="76.2"/>
+<label x="-20.32" y="81.28" size="1.778" layer="95" rot="R90" xref="yes"/>
+<pinref part="R5" gate="G$1" pin="1"/>
+</segment>
+<segment>
+<pinref part="IC1" gate="G$1" pin="A0"/>
+<wire x1="50.8" y1="10.16" x2="55.88" y2="10.16" width="0.1524" layer="91"/>
+<label x="55.88" y="10.16" size="1.778" layer="95" xref="yes"/>
+</segment>
+</net>
+<net name="RIRQ" class="0">
+<segment>
+<pinref part="NRF24L01+" gate="G$1" pin="8"/>
+<wire x1="139.7" y1="2.54" x2="144.78" y2="2.54" width="0.1524" layer="91"/>
+<wire x1="144.78" y1="2.54" x2="144.78" y2="-2.54" width="0.1524" layer="91"/>
+<wire x1="144.78" y1="-2.54" x2="152.4" y2="-2.54" width="0.1524" layer="91"/>
+<label x="152.4" y="-2.54" size="1.778" layer="95" xref="yes"/>
+</segment>
+<segment>
+<pinref part="IC1" gate="G$1" pin="D2"/>
+<wire x1="10.16" y1="17.78" x2="5.08" y2="17.78" width="0.1524" layer="91"/>
+<wire x1="5.08" y1="17.78" x2="5.08" y2="20.32" width="0.1524" layer="91"/>
+<wire x1="5.08" y1="20.32" x2="2.54" y2="20.32" width="0.1524" layer="91"/>
+<label x="2.54" y="20.32" size="1.778" layer="95" rot="R180" xref="yes"/>
+</segment>
+</net>
+<net name="DHT0" class="0">
+<segment>
+<pinref part="IC1" gate="G$1" pin="D4"/>
+<wire x1="10.16" y1="12.7" x2="5.08" y2="12.7" width="0.1524" layer="91"/>
+<wire x1="5.08" y1="12.7" x2="5.08" y2="10.16" width="0.1524" layer="91"/>
+<wire x1="5.08" y1="10.16" x2="2.54" y2="10.16" width="0.1524" layer="91"/>
+<label x="2.54" y="10.16" size="1.778" layer="95" rot="R180" xref="yes"/>
+</segment>
+</net>
