File: door-sensor/hw/energy_monitor.sch (EAGLE design)
At the start: 10 parts, among them IC1 PRO-MINI

Commit message: did a load of stuff that I can't remember and hadn't committed for a while
Parts:
- removed RDSW: (no value), SparkFun-Connectors:CONN_02
- added C2: 0.47uF, SparkFun-Capacitors:10UF-POLAR-RADIAL-2.5MM-25V-20%
- added C5: 10uF, SparkFun-Capacitors:10UF-0603-6.3V-20%
- added CT: (no value), SparkFun-Connectors:CONN_02
- added D1: 200mA/100V/1V, SparkFun-DiscreteSemi:DIODE-1N4148
- added R3: 300k, SparkFun-Resistors:300KOHM-0603-1/10W-1%
- added R4: 100k, SparkFun-Resistors:100KOHM-HORIZ-1/4W-1%
- added R5: 22, SparkFun-Resistors:22OHM-0603-1/10W-1%
- added R6: 1k, SparkFun-Resistors:1KOHM-0603-1/10W-1%
- added R7, R8: 47k, SparkFun-Resistors:47KOHM-0603-1/10W-1%
- BATT: value (none) -> 4.5v
- R1: value 10k -> 22; device SparkFun-Resistors:10KOHM-HORIZ-1/4W-1% -> SparkFun-Resistors:22OHM-0603-1/10W-1%
Connections:
- removed net DHTDO: DHT22.2, R2.2
- removed net SWO: IC1.D3, R1.2, RDSW.2
- new net BATTO: C2.+, IC1.A0, R3.1, R4.2
- new net N$1: R1.2, R5.2, R6.1
- new net N$2: D1.C, R6.2
- new net N$3: R1.1, R5.1
- new net N$4: C5.1, R7.2, R8.1
- net DHTO: now also DHT22.2, R2.2
- net GND: now also C2.-, C5.2, D1.A, R4.1, R7.1; no longer R1.1
- net VCC: now also R3.2, R8.2; no longer RDSW.1
Other:
- moved on the sheet: R1
